Commit message: updated typo

File: fold_elevator_configure/config/fold_elevator.ros2_control.xacro (robot description, xacro)
@@ -3,78 +3,79 @@
 	<xacro:macro name="fold_elevator_ros2_control" params="name sim can_interface desired_config_update_rate">
 		<ros2_control name="fold_elevator" type="system">
-		<hardware>
-			<xacro:if value="${sim}">
-			<plugin>mock_components/GenericSystem</plugin>
-			</xacro:if>
-			<xacro:unless value="${sim}">
-			<plugin>fold_elevator_hardware_interface/FoldElevatorHardwareInterface</plugin>
-			<param name="can_interface">${can_interface}</param>
-			<param name="desired_config_update_rate">${desired_config_update_rate}</param>
-			</xacro:unless>
-		</hardware>
-		<joint name="joint1">
-			<command_interface name="position"/>
-			<state_interface name="position"/>
-			<state_interface name="velocity"/>
-			<param name="can_id">0x60</param>
-			<param name="gear_ratio">101.0</param>
-			<param name="position_offset">A0CC</param>
-			<param name="max_current">22000</param>
-			<param name="min_current">-22000</param>
-			<param name="position_p">5000</param>
-			<param name="position_d">0</param>
-			<param name="velocity_p">300</param>
-			<param name="velocity_i">250</param>
-			<param name="max_velocity">1.0</param>
-			<param name="min_velocity">-1.0</param>
-		</joint>
-		<joint name="joint2">
-			<command_interface name="position"/>
-			<state_interface name="position"/>
-			<state_interface name="velocity"/>
-			<param name="can_id">0x61</param>
-			<param name="gear_ratio">101.0</param>
-			<param name="position_offset">188D6</param>
-			<param name="max_current">22000</param>
-			<param name="min_current">-22000</param>
-			<param name="position_p">4000</param>
-			<param name="position_d">0</param>
-			<param name="velocity_p">90</param>
-			<param name="velocity_i">200</param>
-			<param name="max_velocity">1.0</param>
-			<param name="min_velocity">-1.0</param>
-		</joint>
-		<joint name="joint3">
-			<command_interface name="position"/>
-			<state_interface name="position"/>
-			<state_interface name="velocity"/>
-			<param name="can_id">0x62</param>
-			<param name="gear_ratio">101.0</param>
-			<param name="position_offset">8052</param>
-			<param name="max_current">22000</param>
-			<param name="min_current">-22000</param>
-			<param name="position_p">4600</param>
-			<param name="position_d">0</param>
-			<param name="velocity_p">300</param>
-			<param name="velocity_i">250</param>
-			<param name="max_velocity">1.0</param>
-			<param name="min_velocity">-1.0</param>
-		</joint>
-		<joint name="joint4">
-			<command_interface name="position"/>
-			<state_interface name="position"/>
-			<state_interface name="velocity"/>
-			<param name="can_id">0x63</param>
-			<param name="gear_ratio">121.0</param>
-			<param name="position_offset">28F7</param>
-			<param name="max_current">13000</param>
-			<param name="min_current">-13000</param>
-			<param name="position_p">5200</param>
-			<param name="position_d">0</param>
-			<param name="velocity_p">1250</param>
-			<param name="velocity_i">1500</param>
-			<param name="max_velocity">10.0</param>
-			<param name="min_velocity">-10.0</param>
-		</joint>
+			<hardware>
+				<xacro:if value="${sim}">
+				<plugin>mock_components/GenericSystem</plugin>
+				</xacro:if>
+				<xacro:unless value="${sim}">
+				<plugin>fold_elevator_hardware_interface/FoldElevatorHardwareInterface</plugin>
+				<param name="can_interface">${can_interface}</param>
+				<param name="desired_config_update_rate">${desired_config_update_rate}</param>
+				</xacro:unless>
+			</hardware>
+			<joint name="joint1">
+				<command_interface name="position"/>
+				<state_interface name="position"/>
+				<state_interface name="velocity"/>
+				<param name="can_id">0x60</param>
+				<param name="gear_ratio">101.0</param>
+				<param name="position_offset">A0CC</param>
+				<param name="max_current">22000</param>
+				<param name="min_current">-22000</param>
+				<param name="position_p">5000</param>
+				<param name="position_d">0</param>
+				<param name="velocity_p">300</param>
+				<param name="velocity_i">250</param>
+				<param name="max_velocity">1.0</param>
+				<param name="min_velocity">-1.0</param>
+			</joint>
+			<joint name="joint2">
+				<command_interface name="position"/>
+				<state_interface name="position"/>
+				<state_interface name="velocity"/>
+				<param name="can_id">0x61</param>
+				<param name="gear_ratio">101.0</param>
+				<param name="position_offset">188D6</param>
+				<param name="max_current">22000</param>
+				<param name="min_current">-22000</param>
+				<!-- <param name="position_p">4000</param>      -->
+				<param name="position_p">5000</param>
+				<param name="position_d">0</param>
+				<param name="velocity_p">90</param>
+				<param name="velocity_i">200</param>
+				<param name="max_velocity">1.0</param>
+				<param name="min_velocity">-1.0</param>
+			</joint>
+			<joint name="joint3">
+				<command_interface name="position"/>
+				<state_interface name="position"/>
+				<state_interface name="velocity"/>
+				<param name="can_id">0x62</param>
+				<param name="gear_ratio">101.0</param>
+				<param name="position_offset">8052</param>
+				<param name="max_current">22000</param>
+				<param name="min_current">-22000</param>
+				<param name="position_p">4600</param>
+				<param name="position_d">0</param>
+				<param name="velocity_p">300</param>
+				<param name="velocity_i">250</param>
+				<param name="max_velocity">1.0</param>
+				<param name="min_velocity">-1.0</param>
+			</joint>
+			<joint name="joint4">
+				<command_interface name="position"/>
+				<state_interface name="position"/>
+				<state_interface name="velocity"/>
+				<param name="can_id">0x63</param>
+				<param name="gear_ratio">121.0</param>
+				<param name="position_offset">28F7</param>
+				<param name="max_current">13000</param>
+				<param name="min_current">-13000</param>
+				<param name="position_p">5200</param>
+				<param name="position_d">0</param>
+				<param name="velocity_p">1250</param>
+				<param name="velocity_i">1500</param>
+				<param name="max_velocity">10.0</param>
+				<param name="min_velocity">-10.0</param>
+			</joint>
 		</ros2_control>
 	</xacro:macro>

Commit message: create V2 fold elevator

File: fold_elevator_configure/config/fold_elevator.ros2_control.xacro (robot description, xacro)
@@ -5,10 +5,10 @@
 			<hardware>
 				<xacro:if value="${sim}">
-				<plugin>mock_components/GenericSystem</plugin>
+					<plugin>mock_components/GenericSystem</plugin>
 				</xacro:if>
 				<xacro:unless value="${sim}">
-				<plugin>fold_elevator_hardware_interface/FoldElevatorHardwareInterface</plugin>
-				<param name="can_interface">${can_interface}</param>
-				<param name="desired_config_update_rate">${desired_config_update_rate}</param>
+					<plugin>fold_elevator_hardware_interface/FoldElevatorHardwareInterface</plugin>
+					<param name="can_interface">${can_interface}</param>
+					<param name="desired_config_update_rate">${desired_config_update_rate}</param>
 				</xacro:unless>
 			</hardware>

File: fold_elevator_configure/config/fold_elevator_demo.urdf.xacro (robot description, xacro)
@@ -1,10 +1,10 @@
 <?xml version="1.0"?>
 <robot xmlns:xacro="http://www.ros.org/wiki/xacro" name="fold_elevator">
-    <xacro:include filename="$(find fold_elevator_description)/urdf/fold_elevator.urdf.xacro" />
-    <xacro:include filename="$(find fold_elevator_configure)/config/fold_elevator.ros2_control.xacro" />
-    <link name="world"/>
-    <xacro:fold_elevator name="fold_elevator" parent="world">
-        <origin xyz="0.5 0.5 0.5" rpy="0 0 0"/>
-    </xacro:fold_elevator>
-    <xacro:fold_elevator_ros2_control name="" sim="true" can_interface="can1"/>
+  <xacro:include filename="$(find fold_elevator_description)/urdf/fold_elevator.urdf.xacro" />
+  <xacro:include filename="$(find fold_elevator_configure)/config/fold_elevator.ros2_control.xacro" />
+  <link name="world"/>
+  <xacro:fold_elevator name="fold_elevator" parent="world">
+    <origin xyz="0.0 0.0 0.0" rpy="0 0 0"/>
+  </xacro:fold_elevator>
+  <xacro:fold_elevator_ros2_control name="" sim="true" can_interface="can2" desired_config_update_rate="1000" />
 </robot>

File: fold_elevator_description/urdf/fold_elevator.urdf.xacro (robot description, xacro)
@@ -4,27 +4,30 @@
     <link name="${name}_base_link">
       <inertial>
-        <origin xyz="0.049999 0.056993 0.075571" rpy="0 0 0" />
-        <mass value="0.6213" />
-        <inertia
-          ixx="0.00097836"
-          ixy="4.1808E-09"
-          ixz="1.4286E-08"
-          iyy="0.0010488"
-          iyz="-9.0552E-05"
-          izz="0.00084789" />
-      </inertial>
-      <visual>
-        <origin xyz="0 0 0" rpy="0 0 0" />
-        <geometry>
-          <mesh filename="package://fold_elevator_description/meshes/visual/base_link.STL" scale="0.001 0.001 0.001" />
-        </geometry>
-        <material name="">
-          <color rgba="0.72941 0.74902 0.74902 1.0" />
-        </material>
-      </visual>
-      <collision>
-        <origin xyz="0 0 0" rpy="0 0 0" />
-        <geometry>
-          <mesh filename="package://fold_elevator_description/meshes/collision/base_link.STL" scale="0.001 0.001 0.001" />
+        <origin
+          xyz="0.0891357515039702 -0.0600105188224723 0.0319343260117339"
+          rpy="0 0 0" />
+        <mass
+          value="2.26283180383215" />
+        <inertia
+          ixx="0.00682098629888102"
+          ixy="1.35383918129792E-06"
+          ixz="-0.00120985513326378"
+          iyy="0.00688180551407474"
+          iyz="-3.55019811213944E-06"
+          izz="0.00613738161557863" />
+      </inertial>
+      <visual>
+        <origin xyz="0 0 0" rpy="0 0 0" />
+        <geometry>
+          <mesh filename="package://fold_elevator_description/meshes/visual/base_link.STL" />
+        </geometry>
+        <material name="">
+          <color rgba="0.752941176470588 0.752941176470588 0.752941176470588 1" />
+        </material>
+      </visual>
+      <collision>
+        <origin xyz="0 0 0" rpy="0 0 0" />
+        <geometry>
+          <mesh filename="package://fold_elevator_description/meshes/collision/base_link.STL" />
         </geometry>
       </collision>
@@ -38,35 +41,38 @@
     <link name="link1">
       <inertial>
-        <origin xyz="6.9932E-07 0.24068 -0.05991" rpy="0 0 0" />
-        <mass value="0.76492" />
-        <inertia
-          ixx="0.0065309"
-          ixy="3.0624E-09"
-          ixz="-2.2651E-08"
-          iyy="0.00090992"
-          iyz="6.7991E-05"
-          izz="0.0064905" />
-      </inertial>
-      <visual>
-        <origin xyz="0 0 0" rpy="0 0 0" />
-        <geometry>
-          <mesh filename="package://fold_elevator_description/meshes/visual/link1.STL" scale="0.001 0.001 0.001" />
-        </geometry>
-        <material name="">
-          <color rgba="0.72941 0.74902 0.74902 1" />
-        </material>
-      </visual>
-      <collision>
-        <origin xyz="0 0 0" rpy="0 0 0" />
-        <geometry>
-          <mesh filename="package://fold_elevator_description/meshes/collision/link1.STL" scale="0.001 0.001 0.001" />
+        <origin
+          xyz="0.150849204106985 -9.1876604810387E-06 -0.0581278906888667"
+          rpy="0 0 0" />
+        <mass
+          value="2.976039924942" />
+        <inertia
+          ixx="0.00314898163070912"
+          ixy="1.59802506736583E-06"
+          ixz="-0.00103470671766679"
+          iyy="0.0456464411263901"
+          iyz="-2.66237977525087E-06"
+          izz="0.0473958313229646" />
+      </inertial>
+      <visual>
+        <origin xyz="0 0 0" rpy="0 0 0" />
+        <geometry>
+          <mesh filename="package://fold_elevator_description/meshes/visual/link1.STL" />
+        </geometry>
+        <material name="">
+          <color rgba="0.752941176470588 0.752941176470588 0.752941176470588 1" />
+        </material>
+      </visual>
+      <collision>
+        <origin xyz="0 0 0" rpy="0 0 0" />
+        <geometry>
+          <mesh filename="package://fold_elevator_description/meshes/collision/link1.STL" />
         </geometry>
       </collision>
     </link>
     <joint name="joint1" type="revolute">
-      <origin xyz="0.05 -0.0104 0.1045" rpy="1.57079632679 0 0" />
+      <origin xyz="0.054623 -0.06 0.105" rpy="1.57079632679 -1.57079632679 -1.57079632679" />
       <parent link="${name}_base_link" />
       <child link="link1" />
-      <axis xyz="0 0 -1" />
+      <axis xyz="0 0 1" />
       <limit
         lower="0"
@@ -77,35 +83,38 @@
     <link name="link2">
       <inertial>
-        <origin xyz="-0.00019459 0.23103 -0.088288" rpy="0 0 0" />
-        <mass value="0.77213" />
-        <inertia
-          ixx="0.0065937"
-          ixy="-2.2207E-08"
-          ixz="1.5389E-07"
-          iyy="0.00054292"
-          iyz="-2.341E-05"
-          izz="0.006827" />
-      </inertial>
-      <visual>
-        <origin xyz="0 0 0" rpy="0 0 0" />
-        <geometry>
-          <mesh filename="package://fold_elevator_description/meshes/visual/link2.STL" scale="0.001 0.001 0.001" />
-        </geometry>
-        <material name="">
-          <color rgba="0.72941 0.74902 0.74902 1" />
-        </material>
-      </visual>
-      <collision>
-        <origin xyz="0 0 0" rpy="0 0 0" />
-        <geometry>
-          <mesh filename="package://fold_elevator_description/meshes/collision/link2.STL" scale="0.001 0.001 0.001" />
+        <origin
+          xyz="0.161224779586109 8.26876809245647E-06 -0.00983121345856443"
+          rpy="0 0 0" />
+        <mass
+          value="0.393142489079521" />
+        <inertia
+          ixx="0.000385544833741543"
+          ixy="-2.63936177834169E-09"
+          ixz="-3.85228060816533E-05"
+          iyy="0.00680577641372018"
+          iyz="-1.06477904379006E-11"
+          izz="0.00713642342666465" />
+      </inertial>
+      <visual>
+        <origin xyz="0 0 0" rpy="0 0 0" />
+        <geometry>
+          <mesh filename="package://fold_elevator_description/meshes/visual/link2.STL" />
+        </geometry>
+        <material name="">
+          <color rgba="0.752941176470588 0.752941176470588 0.752941176470588 1" />
+        </material>
+      </visual>
+      <collision>
+        <origin xyz="0 0 0" rpy="0 0 0" />
+        <geometry>
+          <mesh filename="package://fold_elevator_description/meshes/collision/link2.STL" />
         </geometry>
       </collision>
     </link>
     <joint name="joint2" type="revolute">
-      <origin xyz="0 0.325 0.0242" rpy="0 0 0" />
+      <origin xyz="0.325 0 0" rpy="0 0 0" />
       <parent link="link1" />
       <child link="link2" />
-      <axis xyz="0 0 -1" />
+      <axis xyz="0 0 1" />
       <limit
         lower="-2.7925268032"
@@ -116,32 +125,35 @@
     <link name="link3">
       <inertial>
-        <origin xyz="-0.012564 0.064349 -0.0705" rpy="0 0 0" />
-        <mass value="0.2939" />
-        <inertia
-          ixx="0.0012875"
-          ixy="-1.4361E-05"
-          ixz="-5.9979E-07"
-          iyy="0.00054996"
-          iyz="-9.7816E-05"
-          izz="0.0011859" />
-      </inertial>
-      <visual>
-        <origin xyz="0 0 0" rpy="0 0 0" />
-        <geometry>
-          <mesh filename="package://fold_elevator_description/meshes/visual/link3.STL" scale="0.001 0.001 0.001" />
-        </geometry>
-        <material name="">
-          <color rgba="0.69804 0.69804 0.69804 1" />
-        </material>
-      </visual>
-      <collision>
-        <origin xyz="0 0 0" rpy="0 0 0" />
-        <geometry>
-          <mesh filename="package://fold_elevator_description/meshes/collision/link3.STL" scale="0.001 0.001 0.001" />
+        <origin
+          xyz="9.75482671417005E-07 -0.053417702239025 -0.00442438411320098"
+          rpy="0 0 0" />
+        <mass
+          value="0.236077153637359" />
+        <inertia
+          ixx="0.00154414234187567"
+          ixy="-3.0605171029781E-07"
+          ixz="-7.56364769224484E-08"
+          iyy="0.000440001934114007"
+          iyz="-3.94550247420016E-05"
+          izz="0.00123808020961714" />
+      </inertial>
+      <visual>
+        <origin xyz="0 0 0" rpy="0 0 0" />
+        <geometry>
+          <mesh filename="package://fold_elevator_description/meshes/visual/link3.STL" />
+        </geometry>
+        <material name="">
+          <color rgba="0.752941176470588 0.752941176470588 0.752941176470588 1" />
+        </material>
+      </visual>
+      <collision>
+        <origin xyz="0 0 0" rpy="0 0 0" />
+        <geometry>
+          <mesh filename="package://fold_elevator_description/meshes/collision/link3.STL" />
         </geometry>
       </collision>
     </link>
     <joint name="joint3" type="revolute">
-      <origin xyz="0 0.325 0" rpy="0 0 0" />
+      <origin xyz="0.325 0 0" rpy="0 0 1.57079632679" />
       <parent link="link2" />
       <child link="link3" />
@@ -155,32 +167,35 @@
     <link name="link4">
       <inertial>
-        <origin xyz="1.3336E-05 -6.5521E-05 -0.0057552" rpy="0 0 0" />
-        <mass value="0.076276" />
-        <inertia
-          ixx="7.0947E-05"
-          ixy="2.2623E-08"
-          ixz="6.6182E-09"
-          iyy="7.0793E-05"
-          iyz="-4.6063E-08"
-          izz="0.00013988" />
-      </inertial>
-      <visual>
-        <origin xyz="0 0 0" rpy="0 0 0" />
-        <geometry>
-          <mesh filename="package://fold_elevator_description/meshes/visual/link4.STL" scale="0.001 0.001 0.001" />
-        </geometry>
-        <material name="">
-          <color rgba="0.88627 0.88627 0.88627 1" />
-        </material>
-      </visual>
-      <collision>
-        <origin xyz="0 0 0" rpy="0 0 0" />
-        <geometry>
-          <mesh filename="package://fold_elevator_description/meshes/collision/link4.STL" scale="0.001 0.001 0.001" />
+        <origin
+          xyz="-7.51764107198181E-05 -6.84269468244347E-06 -0.00630278043796051"
+          rpy="0 0 0" />
+        <mass
+          value="0.224129183175339" />
+        <inertia
+          ixx="0.000213048176718895"
+          ixy="-8.46287520238891E-08"
+          ixz="-1.96952804294215E-07"
+          iyy="0.000213730397858472"
+          iyz="-2.37665947796012E-08"
+          izz="0.000419496066447268" />
+      </inertial>
+      <visual>
+        <origin xyz="0 0 0" rpy="0 0 0" />
+        <geometry>
+          <mesh filename="package://fold_elevator_description/meshes/visual/link4.STL" />
+        </geometry>
+        <material name="">
+          <color rgba="0.752941176470588 0.752941176470588 0.752941176470588 1" />
+        </material>
+      </visual>
+      <collision>
+        <origin xyz="0 0 0" rpy="0 0 0" />
+        <geometry>
+          <mesh filename="package://fold_elevator_description/meshes/collision/link4.STL" />
         </geometry>
       </collision>
     </link>
     <joint name="joint4" type="revolute">
-      <origin xyz="0 0.1687 -0.07995" rpy="-1.57079632679 0 0" />
+      <origin xyz="0 -0.172 -0.0070273" rpy="1.57079632679 1.57079632679 0" />
       <parent link="link3" />
       <child link="link4" />
